File: mcu.kicad_sch (KiCad schematic)
At the start: 19 parts, among them J301 SWD, SW301 Reset, U301 STM32L053R8T6, Y301 Crystal

Commit message: Updated readme and media
Parts:
- added PA15, PB0, PB1, PB2, PC10, PC11, PC12, PC5: TestPoint_Alt, TestPoint:TestPoint_Pad_D1.0mm, symbol Connector:TestPoint_Alt
Connections:
- net at U301.25 (PC5): now also PC5.1
- net at U301.26 (PB0): now also PB0.1
- net at U301.27 (PB1): now also PB1.1
- net at U301.28 (PB2): now also PB2.1
- net at U301.50 (PA15): now also PA15.1
- net at U301.51 (PC10): now also PC10.1
- net at U301.52 (PC11): now also PC11.1
- net at U301.53 (PC12): now also PC12.1
- no-connect marks 39 -> 31
