File: sniffRF.kicad_pcb (KiCad board)
At the start: 4 copper layers, 113.8 x 23.3 mm, 74 parts, among them J201 USBC, J301 SWD, J401 Ant, J501 FFC_Hirose_FH12-30S-0.5SH_55_, Q501 PMOS, Q502 NMOS, SW301 Reset, U201 BQ24074RGTRG4, U202 MAX17048G+T10, U203 TPS62840DLCR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

Commit message: Updated readme and media
Parts:
- added PA15: TestPoint_Alt, TestPoint:TestPoint_Pad_D1.0mm, F.Cu at (67.9, 42.1)
- added PB0: TestPoint_Alt, TestPoint:TestPoint_Pad_D1.0mm, F.Cu at (75.8, 31.8)
- added PB1: TestPoint_Alt, TestPoint:TestPoint_Pad_D1.0mm, F.Cu at (77.2, 31.8)
- added PB2: TestPoint_Alt, TestPoint:TestPoint_Pad_D1.0mm, F.Cu at (82.5, 32.0)
- added PC10: TestPoint_Alt, TestPoint:TestPoint_Pad_D1.0mm, F.Cu at (68.3, 43.3)
- added PC11: TestPoint_Alt, TestPoint:TestPoint_Pad_D1.0mm, F.Cu at (68.8, 44.6)
- added PC12: TestPoint_Alt, TestPoint:TestPoint_Pad_D1.0mm, F.Cu at (69.4, 45.7)
- added PC5: TestPoint_Alt, TestPoint:TestPoint_Pad_D1.0mm, F.Cu at (83.5, 33.0)
- R505: value 910kΩ -> 620kΩ
Connections:
- net /UI/NC renamed /UI/NC7
- H101 pad 1: Mech_Anchor_3 -> (no net)
- H101 pad 2: Mech_Anchor_3 -> (no net)
- H101 pad 3: Mech_Anchor_3 -> (no net)
- H101 pad 4: Mech_Anchor_3 -> (no net)
- H101 pad 5: Mech_Anchor_3 -> (no net)
- H101 pad 6: Mech_Anchor_3 -> (no net)
- H101 pad 7: Mech_Anchor_3 -> (no net)
- H101 pad 8: Mech_Anchor_3 -> (no net)
- H102 pad 1: Mech_Anchor_4 -> (no net)
- H102 pad 2: Mech_Anchor_4 -> (no net)
- H102 pad 3: Mech_Anchor_4 -> (no net)
- H102 pad 4: Mech_Anchor_4 -> (no net)
- H102 pad 5: Mech_Anchor_4 -> (no net)
- H102 pad 6: Mech_Anchor_4 -> (no net)
- H102 pad 7: Mech_Anchor_4 -> (no net)
- H102 pad 8: Mech_Anchor_4 -> (no net)
- H103 pad 1: Mech_Anchor_1 -> (no net)
- H103 pad 2: Mech_Anchor_1 -> (no net)
- H103 pad 3: Mech_Anchor_1 -> (no net)
- H103 pad 4: Mech_Anchor_1 -> (no net)
- H103 pad 5: Mech_Anchor_1 -> (no net)
- H103 pad 6: Mech_Anchor_1 -> (no net)
- H103 pad 7: Mech_Anchor_1 -> (no net)
- H103 pad 8: Mech_Anchor_1 -> (no net)
- H104 pad 1: Mech_Anchor_2 -> (no net)
- H104 pad 2: Mech_Anchor_2 -> (no net)
- H104 pad 3: Mech_Anchor_2 -> (no net)
- H104 pad 4: Mech_Anchor_2 -> (no net)
- H104 pad 5: Mech_Anchor_2 -> (no net)
- H104 pad 6: Mech_Anchor_2 -> (no net)
- H104 pad 7: Mech_Anchor_2 -> (no net)
- H104 pad 8: Mech_Anchor_2 -> (no net)
- J501 pad 10: GNDREF -> /UI/NC21
- J501 pad 14: GNDREF -> /UI/NC17
- J501 pad 15: GNDREF -> /UI/NC16
- J501 pad 19: GNDREF -> /UI/NC12
- J501 pad 6: GNDREF -> /UI/NC25
- J501 pad 7: GNDREF -> /UI/NC24
- J501 pad 8: GNDREF -> /UI/NC23
- J501 pad 9: GNDREF -> /UI/NC22
- U301 pad 25: unconnected-(U301-PC5-Pad25) -> Net-(U301-PC5)
- U301 pad 26: unconnected-(U301-PB0-Pad26) -> Net-(U301-PB0)
- U301 pad 27: unconnected-(U301-PB1-Pad27) -> Net-(U301-PB1)
- U301 pad 28: unconnected-(U301-PB2-Pad28) -> Net-(U301-PB2)
- U301 pad 50: unconnected-(U301-PA15-Pad50) -> Net-(U301-PA15)
- U301 pad 51: unconnected-(U301-PC10-Pad51) -> Net-(U301-PC10)
- U301 pad 52: unconnected-(U301-PC11-Pad52) -> Net-(U301-PC11)
- U301 pad 53: unconnected-(U301-PC12-Pad53) -> Net-(U301-PC12)
Routing:
- net GNDREF: track 118.8 -> 103.7 mm, vias 105 -> 97
- net Net-(U301-PB0): track 0.00 -> 8.77 mm
- net Net-(U301-PB1): track 0.00 -> 7.22 mm
- net Net-(U301-PB2): track 0.00 -> 4.11 mm
- net Net-(U301-PC5): track 0.00 -> 4.05 mm
- net Net-(U301-PC12): track 0.00 -> 3.72 mm
- net Net-(U301-PC11): track 0.00 -> 3.08 mm
- net Net-(U301-PA15): track 0.00 -> 2.84 mm
- net Net-(U301-PC10): track 0.00 -> 2.84 mm
- net unconnected-(U301-PC12-Pad53): track 1.70 -> 0.00 mm
- net unconnected-(U301-PC10-Pad51): track 1.70 -> 0.00 mm
- net unconnected-(U301-PC5-Pad25): track 1.70 -> 0.00 mm
- net unconnected-(U301-PA15-Pad50): track 1.69 -> 0.00 mm
- net unconnected-(U301-PB2-Pad28): track 1.69 -> 0.00 mm
- net unconnected-(U301-PC11-Pad52): track 1.69 -> 0.00 mm
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Other:
- board text added: "+"
- board text added: "-"
- board text added: "18650"
