File: ui.kicad_sch (KiCad schematic)
At the start: 14 parts, among them J501 FFC_Hirose_FH12-30S-0.5SH_55_, Q501 PMOS, Q502 NMOS

Commit message: Updated readme and file structure, bug fixes and prep for manuf
Parts:
- Q502: LCSC PN C24855 -> C241804
Changed lines of the file:
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@@
 			)
 		)
-		(property "LCSC PN" "C24855"
+		(property "LCSC PN" "C241804"
 			(at 171.45 80.01 0)
 			(effects

Commit message: Updated readme and media
Parts:
- R505: value 910kΩ -> 620kΩ; LCSC PN C3921007 -> C137952; MPN RE0402BRE07910KL -> RC0402FR-07620KL
Connections:
- net GNDREF: no longer J501.10, J501.14, J501.15, J501.19, J501.6, J501.7, J501.8, J501.9
- net NC renamed NC7
- new net NC12: J501.19
- new net NC16: J501.15
- new net NC17: J501.14
- new net NC21: J501.10
- new net NC22: J501.9
- new net NC23: J501.8
- new net NC24: J501.7
- new net NC25: J501.6
- no-connect marks 2 -> 10
Other:
- note added: "OLED Module HS96F04WF C5139756"
- note removed: "OLED Module Wisevision N096-2864KSWEG01-H30 C2890596"
